File: limousine-plate/limousine-plate.kicad_pcb (KiCad board)
At the start: 2 copper layers, 234.4 x 67.9 mm, 0 parts

Commit message: update production files used in v1 run
Other:
- board size 234.4 x 67.9 mm -> 312.5 x 90.5 mm
